File: kicad/usb_voltage_current.sch (KiCad schematic (older format))
At the start: 20 parts, among them J1 Conn_01x01, J10 Conn_01x01, J11 Conn_01x01, J12 Conn_01x01, J13 Conn_01x01, J14 Conn_01x01, J2 Conn_01x01, J3 Conn_01x01, J4 Conn_01x01, J5 Conn_01x01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

Commit message: プルアップ抵抗位置の修正とXIAOのVdd抜け修正
Connections:
- wire segments 53 -> 55
Changed lines of the file:
@@
 EESchema Schematic File Version 4
-LIBS:usb_voltage_current-cache
 EELAYER 29 0
 EELAYER END
@@
 	5600 2350 5700 2350
 Wire Wire Line
-	4050 1800 5600 1800
-Wire Wire Line
 	3950 2300 4100 2300
 Wire Wire Line
 	4100 2300 4100 1750
-Wire Wire Line
-	4100 1750 4300 1750
 Wire Wire Line
 	5550 1750 5550 2250
@@
 	2300 2450 1650 2450
 Wire Wire Line
-	2300 2600 2050 2600
-Wire Wire Line
-	2300 2750 2150 2750
+	2300 2600 2250 2600
 Wire Wire Line
 	2050 2900 2300 2900
@@
 	4300 1250 4300 1300
 Wire Wire Line
+	4950 1200 4950 1250
+Wire Wire Line
+	4950 1250 5200 1250
+Wire Wire Line
+	5200 1250 5200 1300
+Connection ~ 4950 1250
+Wire Wire Line
+	4950 1250 4950 1300
+Wire Wire Line
+	4050 1800 4950 1800
+Wire Wire Line
+	4100 1750 4300 1750
+Wire Wire Line
 	4300 1600 4300 1750
 Connection ~ 4300 1750
@@
 Connection ~ 4550 1750
 Wire Wire Line
-	4550 1750 4950 1750
-Wire Wire Line
-	4950 1200 4950 1250
-Wire Wire Line
-	4950 1250 5200 1250
-Wire Wire Line
-	5200 1250 5200 1300
-Connection ~ 4950 1250
-Wire Wire Line
-	4950 1250 4950 1300
-Wire Wire Line
-	4950 1600 4950 1750
-Connection ~ 4950 1750
-Wire Wire Line
-	4950 1750 5200 1750
-Wire Wire Line
-	5200 1600 5200 1750
-Connection ~ 5200 1750
-Wire Wire Line
-	5200 1750 5550 1750
+	4550 1750 5550 1750
+Wire Wire Line
+	4950 1600 4950 1800
+Connection ~ 4950 1800
+Wire Wire Line
+	4950 1800 5200 1800
+Wire Wire Line
+	5200 1600 5200 1800
+Connection ~ 5200 1800
+Wire Wire Line
+	5200 1800 5600 1800
+$Comp
+L power:+3V3 #PWR08
+U 1 1 5F52972F
+P 2250 1750
+F 0 "#PWR08" H 2250 1600 50  0001 C CNN
+F 1 "+3V3" H 2265 1923 50  0000 C CNN
+F 2 "" H 2250 1750 50  0001 C CNN
+F 3 "" H 2250 1750 50  0001 C CNN
+	1    2250 1750
+	1    0    0    -1
+$EndComp
+Wire Wire Line
+	2300 2750 2150 2750
+Wire Wire Line
+	2250 1750 2250 2600
+Connection ~ 2250 2600
+Wire Wire Line
+	2250 2600 2050 2600
 $EndSCHEMATC

Commit message: なんか変わった
Parts:
- U2: footprint ina226:ina226 -> kicad_mylib:ina226; symbol ina226:INA226 -> usb_voltage_current-rescue:INA226-ina226
Changed lines of the file:
@@
 EESchema Schematic File Version 4
+LIBS:usb_voltage_current-cache
 EELAYER 29 0
 EELAYER END
@@
 NoConn ~ 5700 2550
 $Comp
-L ina226:INA226 U2
+L usb_voltage_current-rescue:INA226-ina226 U2
 U 1 1 5F26533B
 P 5700 2650
 F 0 "U2" H 6228 2976 50  0000 L CNN
 F 1 "INA226" H 6228 2885 50  0000 L CNN
-F 2 "ina226:ina226" H 6300 3250 50  0001 C CNN
+F 2 "kicad_mylib:ina226" H 6300 3250 50  0001 C CNN
 F 3 "" H 6300 3250 50  0001 C CNN
 	1    5700 2650
